Commit message: Changed Duckiebot model

File: catkin_ws/src/duckietown_description/urdf/duckiebot.urdf.xacro (robot description, xacro)
@@ -4,5 +4,5 @@
     <link name="duckiebot">
         <visual>
-            <origin xyz="0 0 0.04" rpy="0 0 ${pi}"/>
+            <origin xyz="0 0 0" rpy="0 0 0"/>
             <geometry>
                 <mesh filename="package://duckietown_description/urdf/meshes/duckiebot.dae" />
