Commit message: adds new tags

File: catkin_ws/src/duckietown_description/urdf/macros.urdf.xacro (robot description, xacro)
@@ -25,5 +25,5 @@
         <link name="tag_${id}">
             <visual>
-                <origin xyz="-0.0254 -0.0254 0" />
+                <origin xyz="0 0 0" />
                 <geometry>
                     <mesh filename="package://duckietown_description/urdf/meshes/tags/tag_${id}.dae" />
